Commit message: update

File: rob10/urdf/iiwa_setup.urdf.xacro (robot description, xacro)
@@ -132,5 +132,5 @@
     <parent link="iiwa_link_ee"/>
     <child link="s_connector_plate"/>
-    <origin xyz="0 0 0" rpy="0 -1.57079 0"/>
+    <origin xyz="0 0 0" rpy="0 -1.57079 1.57079"/>
   </joint>
 </robot>

Commit message: updates

File: rob10/urdf/iiwa_setup.urdf.xacro (robot description, xacro)
@@ -76,5 +76,5 @@
   <xacro:include filename="$(find rob10)/urdf/_d435.urdf.xacro"/>
   <xacro:sensor_d435 parent="camera_ptu_link" prefix="ptu_">
-    <origin xyz="0 0 0" rpy="0 0 0" />
+    <origin xyz="0 0 0" rpy="0 0.0425 0" />
   </xacro:sensor_d435>
   <link name="connector_box_camera">
@@ -83,5 +83,5 @@
         <box size="0.05 0.05 0.05"/>
       </geometry>
-      <origin rpy="0 0 0" xyz="0 0 0.0"/>
+      <origin rpy="0 0 0" xyz="0 0 0"/>
     </visual>
     <collision>

Commit message: more updates

File: rob10/urdf/iiwa_setup.urdf.xacro (robot description, xacro)
@@ -76,5 +76,5 @@
   <xacro:include filename="$(find rob10)/urdf/_d435.urdf.xacro"/>
   <xacro:sensor_d435 parent="camera_ptu_link" prefix="ptu_">
-    <origin xyz="0 0 0" rpy="0 0.0425 0" />
+    <origin xyz="0 0 0" rpy="0 0.04 0" />
   </xacro:sensor_d435>
   <link name="connector_box_camera">

Commit message: More update to the scanner processing node

File: rob10/urdf/iiwa_setup.urdf.xacro (robot description, xacro)
@@ -32,4 +32,25 @@
     <child link="table"/>
     <origin xyz="0 0 0.5" rpy="0 0 0"/>
+  </joint>
+  <!-- SCANNER  -->
+  <link name="laser">
+    <visual>
+      <geometry>
+        <box size="0.06 0.06 0.06"/>
+      </geometry>
+      <origin rpy="0 0 0" xyz="0 0 0.0"/>
+      <material name="aluminum"/>
+    </visual>
+    <collision>
+      <geometry>
+        <box size="0.06 0.06 0.06"/>
+      </geometry>
+      <origin rpy="0 0 0" xyz="0 0 0.0"/>
+    </collision>
+  </link>
+  <joint name="table_scanner_joint" type="fixed">
+    <parent link="table"/>
+    <child link="laser"/>
+    <origin xyz="0.43 -0.02 0.475" rpy="0 0 0"/>
   </joint>
   <!-- PTU ZONE + PROTECTIVE ZONE FOR THE PTU POWER CABLE -->

Commit message: Major updates

File: rob10/urdf/iiwa_setup.urdf.xacro (robot description, xacro)
@@ -33,5 +33,5 @@
     <origin xyz="0 0 0.5" rpy="0 0 0"/>
   </joint>
-  <!-- SCANNER  -->
+  <!-- SCANNER  0.43 -0.02 0.475-->
   <link name="laser">
     <visual>
@@ -47,10 +47,10 @@
       </geometry>
       <origin rpy="0 0 0" xyz="0 0 0.0"/>
-    </collision>
+    </collision>-
   </link>
   <joint name="table_scanner_joint" type="fixed">
     <parent link="table"/>
     <child link="laser"/>
-    <origin xyz="0.43 -0.02 0.475" rpy="0 0 0"/>
+    <origin xyz="0.5 -0.02 0.475" rpy="0 0 0"/>
   </joint>
   <!-- PTU ZONE + PROTECTIVE ZONE FOR THE PTU POWER CABLE -->

File: rob10/urdf/robotiq-3f-gripper_articulated.urdf.xacro (robot description, xacro)
@@ -448,5 +448,5 @@
     <parent link="palm"/>
     <child link="right_ee_link"/>
-    <origin xyz="0 0.146 0" rpy="0 0 1.57"/>
+    <origin xyz="0 0.146 0" rpy="1.57 1.57 3.14"/>
   </joint>
   <joint name="s_model_connector" type="fixed">
