Commit message: New moveIt config files

File: rob10/urdf/iiwa_noPtu_setup_v2.urdf.xacro (robot description, xacro)
@@ -34,5 +34,5 @@
   </joint>
   <!-- SCANNER  -->
-  <!--<link name="laser">
+  <link name="laser">
     <visual>
       <geometry>
@@ -52,5 +52,5 @@
     <parent link="table"/>
     <child link="laser"/>
-    <origin xyz="0.43 -0.02 0.475" rpy="0 0 0"/>
+    <origin xyz="0.325 -0.535 0.4" rpy="0 0 -1.57079"/>
   </joint> -->
   <!-- ROBOT PLATE -->
