Commit message: Demo done

File: rob10/urdf/iiwa_noPtu_setup.urdf.xacro (robot description, xacro)
@@ -52,5 +52,5 @@
     <parent link="table"/>
     <child link="laser"/>
-    <origin xyz="0.43 -0.02 0.475" rpy="0 0 0"/>
+    <origin xyz="0.2 -0.02 0.475" rpy="0 0 0"/>
   </joint>
   <!-- ROBOT PLATE -->

File: rob10/urdf/iiwa_noPtu_setup_v2.urdf.xacro (robot description, xacro)
@@ -52,5 +52,5 @@
     <parent link="table"/>
     <child link="laser"/>
-    <origin xyz="0.325 -0.535 0.4" rpy="0 0 -1.57079"/>
+    <origin xyz="0.105 -0.535 0.4" rpy="0 0 -1.57079"/>
   </joint> -->
   <!-- ROBOT PLATE -->
